File: PCB/IoT_PCB_PiPIco_CS401.kicad_pcb (KiCad board)
At the start: 2 copper layers, 7 parts

Commit message: PCB design
Routing:
- net (no net): track 0.00 -> 182.9 mm
- added copper zone on F.Cu, net (none)
Other:
- board outline added: 21 x 51 mm
- board text added: "CS401 PROJECT BOARD V1.1"
- board text added: "D1"
- board text added: "DS1631"
- board text added: "R1"
- board text added: "R2"
- board text added: "R3"
- board text added: "SW1"
- board text added: "U1"
- board text added: "USB PORT"
